File: Voyager20.sch (KiCad schematic (older format))
At the start: 103 parts, among them Q1 Q_NPN_BEC, SW1 SW_Push, U1 ATmega32U2-AU, U2 PRTR5V0U2X, Y1 16MHz

Commit message: Move Usb
Parts:
- C1, C2, C3, C4, C5, C6, CR1, CR2, CR3, CR4: footprint Capacitors_SMD:C_0603 -> Capacitor_SMD:C_0603_1608Metric
- D1, D10, D11, D12, D13, D14, D15, D16, D17, D19, D2, D20, D21, D22, D25, D26, D27, D28, D3, D4, D5, D6, D7, D8: footprint Diodes_SMD:D_SOD-123 -> Diode_SMD:D_SOD-123
- D18, D23, D24, D9: footprint LEDs:LED_WS2812B-PLCC4 -> LED_SMD:LED_WS2812B_PLCC4_5.0x5.0mm_P3.2mm
- F1: footprint Fuse_Holders_and_Fuses:Fuse_SMD1206_Reflow -> Fuse:Fuse_1206_3216Metric
- Q1: footprint TO_SOT_Packages_SMD:SOT-23 -> Package_TO_SOT_SMD:SOT-23
- R1, R10, R11, R12, R13, R14, R15, R16, R17, R18, R19, R2, R20, R21, R22, R23, R24, R25, R26, R27, R28, R29, R3, R30, R31, R4, R5, R6, R7, R8, R9: footprint Resistors_SMD:R_0805 -> Resistor_SMD:R_0805_2012Metric
- U1: footprint Housings_DFN_QFN:QFN-32-1EP_5x5mm_Pitch0.5mm -> Package_DFN_QFN:QFN-32-1EP_5x5mm_P0.5mm_EP3.65x3.65mm; symbol MCU_Microchip_ATmega:ATmega32U2-AU -> Voyager20-rescue:ATmega32U2-AU-MCU_Microchip_ATmega
- Y1: footprint Crystals:Crystal_SMD_3225-4pin_3.2x2.5mm -> Crystal:Crystal_SMD_3225-4Pin_3.2x2.5mm; symbol Device:Crystal_GND24_Small -> Voyager20-rescue:Crystal_GND24_Small-Device
